File: pcb/willihs.kicad_pcb (KiCad board)
At the start: 2 copper layers, 188.9 x 83.9 mm, 114 parts, among them J1 SWD, J2 Battery, J3 USB-C Conn, J4 Pico EZMate, J5 TC2030_SWD, K1 KEYSW, K10 KEYSW, K11 KEYSW, K12 KEYSW, K13 KEYSW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

Commit message: updates
Parts:
- J4: footprint Connector_Molex:Molex_Pico-EZmate_78171-0002_1x02-1MP_P1.20mm_Vertical -> zackforbing:Molex_Pico-EZmate_78171-0002_1x02-1MP_P1.20mm_Vertical reversible
- moved J4 1.97 mm to (204.2, 43.2)
Routing:
- net VBAT: track 33.0 -> 39.0 mm
